File: FrontEnd/hardware/FirstYokePCB/WheelFrontEndDevBoard_PCB.kicad_pcb (KiCad board)
At the start: 4 copper layers, 89.7 x 73.2 mm, 108 parts, among them J1 Programming, J2 CAN, J3 Buttons, J4 RotaryEncoders, J5 Paddels, P1 USB_C_Plug, SW1 Reset, U2 STM32G491VETx, U3 AMS1117-3.3, U4 TCAN332G, U5 MIC2544-2YM, Y1 Crystal_GND24

Commit message: Finished PCB (finished layout)
Parts:
- added H1: MountingHole, MountingHole:MountingHole_3.2mm_M3, F.Cu at (19.9, 88.2)
- added H2: MountingHole, MountingHole:MountingHole_3.2mm_M3, F.Cu at (19.9, 23.0)
- added H3: MountingHole, MountingHole:MountingHole_3.2mm_M3, F.Cu at (101.6, 23.0)
- added H4: MountingHole, MountingHole:MountingHole_3.2mm_M3, F.Cu at (101.6, 88.2)
- D1, D2, D3, D4, D5, D6, D7: moved to F.Cu
- moved TP1 23.2 mm to (38.4, 28.2), turned to 180 degrees
- moved C11 4.58 mm to (51.1, 72.3)
- moved C12 4.58 mm to (49.7, 72.3)
- moved C4 4.58 mm to (46.7, 72.3)
- moved R2 4.58 mm to (48.2, 72.3)
- moved JP2 4.58 mm to (55.0, 73.7)
- moved C7 0.44 mm to (38.7, 71.9)
Connections:
- R24 pad 1: /MCU/PD5/LED1 -> /MCU/PD9/LED1
- R25 pad 1: /MCU/PD6/LED2 -> /MCU/PD8/LED2
- R26 pad 1: /MCU/PD7/LED3 -> /MCU/PD5/LED3
- R27 pad 1: /MCU/PD8/LED4 -> /MCU/PD6/LED4
- R28 pad 1: /MCU/PD9/LED5 -> /MCU/PD7/LED5
- U2 pad 55: /MCU/PD8/LED4 -> /MCU/PD8/LED2
- U2 pad 56: /MCU/PD9/LED5 -> /MCU/PD9/LED1
- U2 pad 82: /MCU/PD0/EncoderA3 -> /MCU/PD3/EncoderB4
- U2 pad 83: /MCU/PD1/EncoderB3 -> /MCU/PD2/EncoderA4
- U2 pad 84: /MCU/PD2/EncoderA4 -> /MCU/PD1/EncoderB3
- U2 pad 85: /MCU/PD3/EncoderB4 -> /MCU/PD0/EncoderA3
- U2 pad 87: /MCU/PD5/LED1 -> /MCU/PD5/LED3
- U2 pad 88: /MCU/PD6/LED2 -> /MCU/PD6/LED4
- U2 pad 89: /MCU/PD7/LED3 -> /MCU/PD7/LED5
Routing:
- net VBUS: track 2.54 -> 94.8 mm, vias 0 -> 2
- net GND: track 0.00 -> 87.5 mm, vias 0 -> 177
- net +3.3V: track 48.3 -> 131.4 mm, vias 0 -> 51
- net /MCU/CAN_TX: track 0.00 -> 76.0 mm
- net /MCU/PD11/Paddel0: track 5.88 -> 80.1 mm, vias 0 -> 2
- net /MCU/CAN_RX: track 0.00 -> 73.2 mm
- net /MCU/PD12/Paddel1: track 5.72 -> 75.9 mm, vias 0 -> 2
- net /MCU/PE0/button0: track 6.51 -> 73.0 mm, vias 0 -> 2
- net /MCU/PD8/LED2: track 0.00 -> 65.1 mm, vias 0 -> 2
- net /MCU/PE1/button1: track 6.35 -> 68.3 mm, vias 0 -> 2
- net /MCU/PD9/LED1: track 0.00 -> 60.1 mm, vias 0 -> 2
- net /MCU/PD10/LED6: track 0.00 -> 55.1 mm, vias 0 -> 2
- net /MCU/PE2/button2: track 6.19 -> 59.6 mm, vias 0 -> 2
- net /MCU/PE3/button3: track 6.04 -> 55.4 mm, vias 0 -> 2
- net /MCU/PE4/button4: track 5.88 -> 52.9 mm, vias 0 -> 2
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- added copper zone on B.Cu, net GND
- added copper zone on F.Cu, net GND
Other:
- board text added: "+3.3V"
- board text added: "+5V"
- board text added: "B9,B8,B7,B6,B5,B4,B3,B2,B1,B0"
- board text added: "CAN_H"
- board text added: "CAN_L"
- board text added: "EncoderA0"
- board text added: "EncoderA1"
- board text added: "EncoderA2"
- board text added: "EncoderA3"
- board text added: "EncoderA4"
- board text added: "EncoderB0"
- board text added: "EncoderB1"
- board text added: "EncoderB2"
- board text added: "EncoderB3"
- board text added: "EncoderB4"
- board text added: "GND"
- board text added: "NRST"
- board text added: "P1,P0"
- board text added: "RPM"
- board text added: "Reset"
- board text added: "SWDCLK"
- board text added: "SWDIO"
- board text added: "VBUS"
