File: FrontEnd/hardware/FirstYokePCB/mcu.kicad_sch (KiCad schematic)
At the start: 108 parts, among them J1 Programming, J2 CAN, J3 Buttons, J4 RotaryEncoders, J5 Paddels, P1 USB_C_Plug, SW1 Reset, U2 STM32G491VETx, U3 AMS1117-3.3, U4 TCAN332G, U5 MIC2544-2YM, Y1 Crystal_GND24

Commit message: Finished PCB (finished layout)
Parts:
- added H1, H2, H3, H4: MountingHole, MountingHole:MountingHole_3.2mm_M3, symbol Mechanical:MountingHole
Connections:
- net PD0/EncoderA3: now also U2.85 (PD3); no longer U2.82 (PD0)
- net PD1/EncoderB3: now also U2.84 (PD2); no longer U2.83 (PD1)
- net PD2/EncoderA4: now also U2.83 (PD1); no longer U2.84 (PD2)
- net PD3/EncoderB4: now also U2.82 (PD0); no longer U2.85 (PD3)
- net PD5/LED1 renamed PD5/LED3
- net PD5/LED3: now also R26.1; no longer R24.1
- net PD6/LED2 renamed PD6/LED4
- net PD6/LED4: now also R27.1; no longer R25.1
- net PD7/LED3 renamed PD7/LED5
- net PD7/LED5: now also R28.1; no longer R26.1
- net PD8/LED4 renamed PD8/LED2
- net PD8/LED2: now also R25.1; no longer R27.1
- net PD9/LED5 renamed PD9/LED1
- net PD9/LED1: now also R24.1; no longer R28.1
